Commit message: update code

File: fet_description/urdf/turtlebot3_fet.urdf.xacro (robot description, xacro)
@@ -14,5 +14,5 @@
       <origin xyz="0 0 0" rpy="0 0 0"/>
       <geometry>
-        <mesh filename="package://fet_description/meshes/bases/waffle_pi_base.stl" scale="0.001 0.001 0.001"/>
+        <mesh filename="package://fet_description/meshes/bases/fet_base.stl" scale="0.001 0.001 0.001"/>
       </geometry>
       <material name="light_black"/>
